Commit message: removed all build files

File: ws/crawler/description/robot_core.xacro (robot description, xacro)
@@ -1,5 +1,11 @@
 <?xml version="1.0"?>
-<robot xmlns:xacro="http://www.ros.org/wiki/xacro" >
+<robot xmlns:xacro="http://www.ros.org/wiki/xacro">
+    <xacro:include filename="inertial_macros.xacro" />
     <link name="base_link">
+        <inertial>
+            <origin xyz="0 0 0" rpy="0 0 0"/>
+            <mass value="1"/>
+            <inertia ixx="0.1" ixy="0" ixz="0" iyy="0.1" iyz="0" izz="0.1"/>
+        </inertial>
     </link>
     <joint name="joint_chassis" type="fixed">
@@ -12,4 +18,7 @@
             <origin xyz="0 0 -0.025" rpy="0 0 0"/>
             <geometry>
+                <!--
+                <box size="0.4 0.4 0.05"/>
+                -->
                 <mesh filename="package://crawler/meshes/chassis.dae" scale="1 1 1" />
             </geometry>
@@ -18,4 +27,15 @@
             </material>
         </visual>
+        <inertial>
+            <origin xyz="0 0 0" rpy="0 0 0"/>
+            <mass value="1"/>
+            <inertia ixx="0.1" ixy="0" ixz="0" iyy="0.1" iyz="0" izz="0.1"/>
+        </inertial>
+        <collision>
+            <origin xyz="0 0 0" rpy="0 0 0"/>
+            <geometry>
+                <box size="0.4 0.4 0.05"/>
+            </geometry>
+        </collision>
     </link>
     <joint name="joint_front_left_wheel" type="continuous">
@@ -24,9 +44,10 @@
         <child link="front_left_wheel"/>
         <axis xyz="1 0 0"/>
+        <mimic joint="joint_center_left_wheel" multiplier="1" offset="0"/>
     </joint>
     <joint name="joint_center_left_wheel" type="continuous">
-        <origin xyz="0.19 0 0" rpy="0 0 0"/>
         <parent link="chassis"/>
         <child link="center_left_wheel"/>
+        <origin xyz="0.19 0 0" rpy="0 0 0"/>
         <axis xyz="1 0 0"/>
     </joint>
@@ -36,4 +57,5 @@
         <child link="back_left_wheel"/>
         <axis xyz="1 0 0"/>
+        <mimic joint="joint_center_left_wheel" multiplier="1" offset="0"/>
     </joint>
     <link name="front_left_wheel">
@@ -44,4 +66,13 @@
             </geometry>
         </visual>
+        <collision>
+            <origin xyz="0 0 0" rpy="0 ${3.141/2} 0"/>
+            <geometry>
+                <cylinder radius="0.0625" length="0.05"/>
+            </geometry>
+        </collision>
+        <xacro:inertial_cylinder mass="0.1" radius="0.0625" length="0.02">
+            <origin xyz="0 0 0" rpy="0 0 0"/>
+        </xacro:inertial_cylinder>
     </link>
     <link name="center_left_wheel">
@@ -52,4 +83,13 @@
             </geometry>
         </visual>
+        <collision>
+            <origin xyz="0 0 0" rpy="0 ${3.141/2} 0"/>
+            <geometry>
+                <cylinder radius="0.0625" length="0.05"/>
+            </geometry>
+        </collision>
+        <xacro:inertial_cylinder mass="0.1" radius="0.0625" length="0.02">
+            <origin xyz="0 0 0" rpy="0 0 0"/>
+        </xacro:inertial_cylinder>
     </link>
     <link name="back_left_wheel">
@@ -60,4 +100,13 @@
             </geometry>
         </visual>
+        <collision>
+            <origin xyz="0 0 0" rpy="0 ${3.141/2} 0"/>
+            <geometry>
+                <cylinder radius="0.0625" length="0.05"/>
+            </geometry>
+        </collision>
+        <xacro:inertial_cylinder mass="0.1" radius="0.0625" length="0.02">
+            <origin xyz="0 0 0" rpy="0 0 0"/>
+        </xacro:inertial_cylinder>
     </link>
     <joint name="joint_front_right_wheel" type="continuous">
@@ -66,4 +115,5 @@
         <child link="front_right_wheel"/>
         <axis xyz="1 0 0"/>
+        <mimic joint="joint_center_right_wheel" multiplier="1" offset="0"/>\
     </joint>
     <joint name="joint_center_right_wheel" type="continuous">
@@ -78,4 +128,5 @@
         <child link="back_right_wheel"/>
         <axis xyz="1 0 0"/>
+        <mimic joint="joint_center_right_wheel" multiplier="1" offset="0"/>
     </joint>
     <link name="front_right_wheel">
@@ -86,4 +137,13 @@
             </geometry>
         </visual>
+        <collision>
+            <origin xyz="0 0 0" rpy="0 ${3.141/2} 0"/>
+            <geometry>
+                <cylinder radius="0.0625" length="0.05"/>
+            </geometry>
+        </collision>
+        <xacro:inertial_cylinder mass="0.1" radius="0.0625" length="0.02">
+            <origin xyz="0 0 0" rpy="0 0 0"/>
+        </xacro:inertial_cylinder>
     </link>
     <link name="center_right_wheel">
@@ -94,4 +154,13 @@
             </geometry>
         </visual>
+        <collision>
+            <origin xyz="0 0 0" rpy="0 ${3.141/2} 0"/>
+            <geometry>
+                <cylinder radius="0.0625" length="0.05"/>
+            </geometry>
+        </collision>
+        <xacro:inertial_cylinder mass="0.1" radius="0.0625" length="0.02">
+            <origin xyz="0 0 0" rpy="0 0 0"/>
+        </xacro:inertial_cylinder>
     </link>
     <link name="back_right_wheel">
@@ -102,4 +171,13 @@
             </geometry>
         </visual>
+        <collision>
+            <origin xyz="0 0 0" rpy="0 ${3.141/2} 0"/>
+            <geometry>
+                <cylinder radius="0.0625" length="0.05"/>
+            </geometry>
+        </collision>
+        <xacro:inertial_cylinder mass="0.1" radius="0.0625" length="0.02">
+            <origin xyz="0 0 0" rpy="0 0 0"/>
+        </xacro:inertial_cylinder>
     </link>
 </robot>

File: ws/crawler/description/ros2_control.xacro (robot description, xacro)
@@ -1,4 +1,5 @@
 <?xml version="1.0"?>
 <robot xmlns:xacro="http://www.ros.org/wiki/xacro">
+    <!--
     <ros2_control name="RealRobot" type="system">
         <hardware>
@@ -7,8 +8,6 @@
             <param name="right_wheel_name">joint_center_right_wheel</param>
             <param name="loop_rate">30</param>
-            <!--
+            <param name="device">/dev/ttyACM0</param>
             <param name="device">/dev/pts/6</param>
-            -->
-            <param name="device">/dev/ttyACM0</param>
             <param name="baud_rate">115200</param>
             <param name="timeout_ms">1000</param>
@@ -33,3 +32,31 @@
         </joint>
     </ros2_control>
+    -->
+    <ros2_control name="GazeboSystem" type="system">
+        <hardware>
+            <plugin>gazebo_ros2_control/GazeboSystem</plugin>
+        </hardware>
+        <joint name="joint_center_left_wheel">
+            <command_interface name="velocity">
+                <param name="min">-10</param>
+                <param name="max">10</param>
+            </command_interface>
+            <state_interface name="position"/>
+            <state_interface name="velocity"/>
+        </joint>
+        <joint name="joint_center_right_wheel">
+            <command_interface name="velocity">
+                <param name="min">-10</param>
+                <param name="max">10</param>
+            </command_interface>
+            <command_interface name="velocity"/>
+            <state_interface name="position"/>
+            <state_interface name="velocity"/>
+        </joint>
+    </ros2_control>
+    <gazebo>
+        <plugin filename="libgazebo_ros2_control.so" name="gazebo_ros2_control">
+        <parameters>$(find crawler)/config/diffbot_controllers.yaml</parameters>
+        </plugin>
+    </gazebo>
 </robot>

Commit message: Added all wheels to be powered and changed friction

File: ws/crawler/description/robot_core.xacro (robot description, xacro)
@@ -181,3 +181,75 @@
         </xacro:inertial_cylinder>
     </link>
+    <gazebo reference="back_right_wheel">
+        <collision>
+            <surface>
+                <friction>
+                    <ode>
+                        <mu>0.1</mu>
+                        <mu2>0.1</mu2>
+                    </ode>
+                </friction>
+            </surface>
+        </collision>
+    </gazebo>
+        <gazebo reference="center_right_wheel">
+        <collision>
+            <surface>
+                <friction>
+                    <ode>
+                        <mu>0.1</mu>
+                        <mu2>0.1</mu2>
+                    </ode>
+                </friction>
+            </surface>
+        </collision>
+    </gazebo>
+        <gazebo reference="front_right_wheel">
+        <collision>
+            <surface>
+                <friction>
+                    <ode>
+                        <mu>0.1</mu>
+                        <mu2>0.1</mu2>
+                    </ode>
+                </friction>
+            </surface>
+        </collision>
+    </gazebo>
+    <gazebo reference="back_left_wheel">
+        <collision>
+            <surface>
+                <friction>
+                    <ode>
+                        <mu>0.1</mu>
+                        <mu2>0.1</mu2>
+                    </ode>
+                </friction>
+            </surface>
+        </collision>
+    </gazebo>
+        <gazebo reference="center_left_wheel">
+        <collision>
+            <surface>
+                <friction>
+                    <ode>
+                        <mu>0.1</mu>
+                        <mu2>0.1</mu2>
+                    </ode>
+                </friction>
+            </surface>
+        </collision>
+    </gazebo>
+        <gazebo reference="front_left_wheel">
+        <collision>
+            <surface>
+                <friction>
+                    <ode>
+                        <mu>0.1</mu>
+                        <mu2>0.1</mu2>
+                    </ode>
+                </friction>
+            </surface>
+        </collision>
+    </gazebo>
 </robot>

File: ws/crawler/description/ros2_control.xacro (robot description, xacro)
@@ -54,8 +54,42 @@
             <state_interface name="velocity"/>
         </joint>
+        <joint name="joint_front_left_wheel">
+            <command_interface name="velocity">
+                <param name="min">-10</param>
+                <param name="max">10</param>
+            </command_interface>
+            <state_interface name="position"/>
+            <state_interface name="velocity"/>
+        </joint>
+        <joint name="joint_front_right_wheel">
+            <command_interface name="velocity">
+                <param name="min">-10</param>
+                <param name="max">10</param>
+            </command_interface>
+            <command_interface name="velocity"/>
+            <state_interface name="position"/>
+            <state_interface name="velocity"/>
+        </joint>
+        <joint name="joint_back_left_wheel">
+            <command_interface name="velocity">
+                <param name="min">-10</param>
+                <param name="max">10</param>
+            </command_interface>
+            <state_interface name="position"/>
+            <state_interface name="velocity"/>
+        </joint>
+        <joint name="joint_back_right_wheel">
+            <command_interface name="velocity">
+                <param name="min">-10</param>
+                <param name="max">10</param>
+            </command_interface>
+            <command_interface name="velocity"/>
+            <state_interface name="position"/>
+            <state_interface name="velocity"/>
+        </joint>
     </ros2_control>
     <gazebo>
         <plugin filename="libgazebo_ros2_control.so" name="gazebo_ros2_control">
-        <parameters>$(find crawler)/config/diffbot_controllers.yaml</parameters>
+        <parameters>$(find crawler)/config/diffbot_controllers_gazebo.yaml</parameters>
         </plugin>
     </gazebo>

Commit message: added livox simulation package as submodule

File: ws/crawler/description/robot_core.xacro (robot description, xacro)
@@ -2,4 +2,5 @@
 <robot xmlns:xacro="http://www.ros.org/wiki/xacro">
     <xacro:include filename="inertial_macros.xacro" />
+    <xacro:include filename="$(find ros2_livox_simulation)/urdf/mid360.xacro" />
     <link name="base_link">
         <inertial>
@@ -253,3 +254,38 @@
         </collision>
     </gazebo>
+    <xacro:mid360 name="livox" parent="base_link" topic="livox/lidar">
+        <origin xyz="0 0 0.1" rpy="0 0 0"/>
+    </xacro:mid360>
+  <joint name="imu_joint" type="fixed">
+        <parent link="chassis"/>
+        <child link="imu"/>
+        <origin xyz="0.055 0 0.175" rpy="0 0 0"/>
+    </joint>
+    <link name="imu">
+        <visual>
+            <geometry>
+                <box size="0.03 0.03 0.03"/>
+            </geometry>
+        </visual>
+    </link>
+  <gazebo reference="imu">
+    <gravity>true</gravity>
+    <sensor name="imu_sensor" type="imu">
+      <always_on>true</always_on>
+      <update_rate>100</update_rate>
+      <visualize>true</visualize>
+      <topic>default_topic</topic>
+      <plugin filename="libgazebo_ros_imu_sensor.so" name="imu_plugin">
+        <topicName>imu</topicName>
+        <bodyName>imu</bodyName>
+        <updateRateHZ>10.0</updateRateHZ>
+        <gaussianNoise>0.0</gaussianNoise>
+        <xyzOffset>0 0 0</xyzOffset>
+        <rpyOffset>0 0 0</rpyOffset>
+        <frameName>imu</frameName>
+        <initial_orientation_as_reference>false</initial_orientation_as_reference>
+      </plugin>
+      <pose>0 0 0 0 0 0</pose>
+    </sensor>
+  </gazebo>
 </robot>

Commit message: added base_footprint and laser links

File: ws/crawler/description/robot_core.xacro (robot description, xacro)
@@ -3,4 +3,5 @@
     <xacro:include filename="inertial_macros.xacro" />
     <xacro:include filename="$(find ros2_livox_simulation)/urdf/mid360.xacro" />
+    <xacro:property name="PI" value="3.1415926"/>
     <link name="base_link">
         <inertial>
@@ -15,4 +16,11 @@
         <child link="chassis"/>
     </joint>
+    <link name='base_footprint'>
+    </link>
+    <joint name="joint_base_footprint" type="fixed">
+        <origin xyz="0 0 0" rpy="0 0 -1.57"/>
+        <parent link="base_link"/>
+        <child link="base_footprint"/>
+    </joint>
     <link name="chassis">
         <visual>
@@ -255,5 +263,5 @@
     </gazebo>
     <xacro:mid360 name="livox" parent="base_link" topic="livox/lidar">
-        <origin xyz="0 0 0.1" rpy="0 0 0"/>
+        <origin xyz="0 0 0.1" rpy="0 0 -1.57"/>
     </xacro:mid360>
   <joint name="imu_joint" type="fixed">
@@ -289,3 +297,10 @@
     </sensor>
   </gazebo>
+    <link name="laser_frame">
+    </link>
+    <joint name="laser_joint" type="fixed">
+        <parent link="chassis"/>
+        <child link="laser_frame"/>
+        <origin xyz="0.1 0 0.1" rpy="0 0 0"/>
+    </joint>
 </robot>

Commit message: removed simulation only macros

File: ws/crawler/description/robot_core.xacro (robot description, xacro)
@@ -2,5 +2,7 @@
 <robot xmlns:xacro="http://www.ros.org/wiki/xacro">
     <xacro:include filename="inertial_macros.xacro" />
-    <xacro:include filename="$(find ros2_livox_simulation)/urdf/mid360.xacro" />
+    <xacro:if value="$(arg sim_mode)">
+        <xacro:include filename="$(find ros2_livox_simulation)/urdf/mid360.xacro" />
+    </xacro:if>
     <xacro:property name="PI" value="3.1415926"/>
     <link name="base_link">
@@ -262,7 +264,9 @@
         </collision>
     </gazebo>
-    <xacro:mid360 name="livox" parent="base_link" topic="livox/lidar">
-        <origin xyz="0 0 0.1" rpy="0 0 -1.57"/>
-    </xacro:mid360>
+    <xacro:if value="$(arg sim_mode)">
+        <xacro:mid360 name="livox" parent="base_link" topic="livox/lidar">
+            <origin xyz="0 0 0.1" rpy="0 0 -1.57"/>
+        </xacro:mid360>
+    </xacro:if>
   <joint name="imu_joint" type="fixed">
         <parent link="chassis"/>

Commit message: Removed rotation of frames as its now handled by fast_lio

File: ws/crawler/description/robot_core.xacro (robot description, xacro)
@@ -266,5 +266,8 @@
     <xacro:if value="$(arg sim_mode)">
         <xacro:mid360 name="livox" parent="base_link" topic="livox/lidar">
+            <!--
             <origin xyz="0 0 0.1" rpy="0 0 -1.57"/>
+            -->
+            <origin xyz="0 0 0.1" rpy="0 0 0"/>
         </xacro:mid360>
     </xacro:if>
