Commit message: Reached (almost) state of diablo/go2 simulations - Added local_planner and its dependencies - Added far_planner and its dependencies - Added tare_planner - Added tool for tracking exploration

File: ws/crawler/description/robot_core.xacro (robot description, xacro)
@@ -10,5 +10,5 @@
             <origin xyz="0 0 0" rpy="0 0 0"/>
             <mass value="1"/>
-            <inertia ixx="0.1" ixy="0" ixz="0" iyy="0.1" iyz="0" izz="0.1"/>
+            <inertia ixx="0.1" ixy="0.1" ixz="0.1" iyy="0.1" iyz="0" izz="0.1"/>
         </inertial>
     </link>
@@ -31,5 +31,5 @@
                 <!--
                 <box size="0.4 0.4 0.05"/>
-                -->
+                -->`
                 <mesh filename="package://crawler/meshes/chassis.dae" scale="1 1 1" />
             </geometry>
@@ -70,18 +70,20 @@
         <mimic joint="joint_center_left_wheel" multiplier="1" offset="0"/>
     </joint>
+    <xacro:property name="wheel_r" value="0.0652"/>
+    <xacro:property name="wheel_l" value="0.03"/>
     <link name="front_left_wheel">
         <visual>
             <origin xyz="0 0 0" rpy="0 ${3.141/2} 0"/>
             <geometry>
-                <cylinder radius="0.0625" length="0.05"/>
-            </geometry>
-        </visual>
-        <collision>
-            <origin xyz="0 0 0" rpy="0 ${3.141/2} 0"/>
-            <geometry>
-                <cylinder radius="0.0625" length="0.05"/>
-            </geometry>
-        </collision>
-        <xacro:inertial_cylinder mass="0.1" radius="0.0625" length="0.02">
+                <cylinder radius="${wheel_r}" length="${wheel_l}"/>
+            </geometry>
+        </visual>
+        <collision>
+            <origin xyz="0 0 0" rpy="0 ${3.141/2} 0"/>
+            <geometry>
+                <cylinder radius="${wheel_r}" length="${wheel_l}"/>
+            </geometry>
+        </collision>
+        <xacro:inertial_cylinder mass="0.1" radius="${wheel_r}" length="${wheel_l}">
             <origin xyz="0 0 0" rpy="0 0 0"/>
         </xacro:inertial_cylinder>
@@ -91,14 +93,14 @@
             <origin xyz="0 0 0" rpy="0 ${3.141/2} 0"/>
             <geometry>
-                <cylinder radius="0.0625" length="0.05"/>
-            </geometry>
-        </visual>
-        <collision>
-            <origin xyz="0 0 0" rpy="0 ${3.141/2} 0"/>
-            <geometry>
-                <cylinder radius="0.0625" length="0.05"/>
-            </geometry>
-        </collision>
-        <xacro:inertial_cylinder mass="0.1" radius="0.0625" length="0.02">
+                <cylinder radius="${wheel_r}" length="${wheel_l}"/>
+            </geometry>
+        </visual>
+        <collision>
+            <origin xyz="0 0 0" rpy="0 ${3.141/2} 0"/>
+            <geometry>
+                <cylinder radius="${wheel_r}" length="${wheel_l}"/>
+            </geometry>
+        </collision>
+        <xacro:inertial_cylinder mass="0.1" radius="${wheel_r}" length="${wheel_l}">
             <origin xyz="0 0 0" rpy="0 0 0"/>
         </xacro:inertial_cylinder>
@@ -108,14 +110,14 @@
             <origin xyz="0 0 0" rpy="0 ${3.141/2} 0"/>
             <geometry>
-                <cylinder radius="0.0625" length="0.05"/>
-            </geometry>
-        </visual>
-        <collision>
-            <origin xyz="0 0 0" rpy="0 ${3.141/2} 0"/>
-            <geometry>
-                <cylinder radius="0.0625" length="0.05"/>
-            </geometry>
-        </collision>
-        <xacro:inertial_cylinder mass="0.1" radius="0.0625" length="0.02">
+                <cylinder radius="${wheel_r}" length="${wheel_l}"/>
+            </geometry>
+        </visual>
+        <collision>
+            <origin xyz="0 0 0" rpy="0 ${3.141/2} 0"/>
+            <geometry>
+                <cylinder radius="${wheel_r}" length="${wheel_l}"/>
+            </geometry>
+        </collision>
+        <xacro:inertial_cylinder mass="0.1" radius="${wheel_r}" length="${wheel_l}">
             <origin xyz="0 0 0" rpy="0 0 0"/>
         </xacro:inertial_cylinder>
@@ -145,14 +147,14 @@
             <origin xyz="0 0 0" rpy="0 ${3.141/2} 0"/>
             <geometry>
-                <cylinder radius="0.0625" length="0.05"/>
-            </geometry>
-        </visual>
-        <collision>
-            <origin xyz="0 0 0" rpy="0 ${3.141/2} 0"/>
-            <geometry>
-                <cylinder radius="0.0625" length="0.05"/>
-            </geometry>
-        </collision>
-        <xacro:inertial_cylinder mass="0.1" radius="0.0625" length="0.02">
+                <cylinder radius="${wheel_r}" length="${wheel_l}"/>
+            </geometry>
+        </visual>
+        <collision>
+            <origin xyz="0 0 0" rpy="0 ${3.141/2} 0"/>
+            <geometry>
+                <cylinder radius="${wheel_r}" length="${wheel_l}"/>
+            </geometry>
+        </collision>
+        <xacro:inertial_cylinder mass="0.1" radius="${wheel_r}" length="${wheel_l}">
             <origin xyz="0 0 0" rpy="0 0 0"/>
         </xacro:inertial_cylinder>
@@ -162,14 +164,14 @@
             <origin xyz="0 0 0" rpy="0 ${3.141/2} 0"/>
             <geometry>
-                <cylinder radius="0.0625" length="0.05"/>
-            </geometry>
-        </visual>
-        <collision>
-            <origin xyz="0 0 0" rpy="0 ${3.141/2} 0"/>
-            <geometry>
-                <cylinder radius="0.0625" length="0.05"/>
-            </geometry>
-        </collision>
-        <xacro:inertial_cylinder mass="0.1" radius="0.0625" length="0.02">
+                <cylinder radius="${wheel_r}" length="${wheel_l}"/>
+            </geometry>
+        </visual>
+        <collision>
+            <origin xyz="0 0 0" rpy="0 ${3.141/2} 0"/>
+            <geometry>
+                <cylinder radius="${wheel_r}" length="${wheel_l}"/>
+            </geometry>
+        </collision>
+        <xacro:inertial_cylinder mass="0.1" radius="${wheel_r}" length="${wheel_l}">
             <origin xyz="0 0 0" rpy="0 0 0"/>
         </xacro:inertial_cylinder>
@@ -179,24 +181,30 @@
             <origin xyz="0 0 0" rpy="0 ${3.141/2} 0"/>
             <geometry>
-                <cylinder radius="0.0625" length="0.05"/>
-            </geometry>
-        </visual>
-        <collision>
-            <origin xyz="0 0 0" rpy="0 ${3.141/2} 0"/>
-            <geometry>
-                <cylinder radius="0.0625" length="0.05"/>
-            </geometry>
-        </collision>
-        <xacro:inertial_cylinder mass="0.1" radius="0.0625" length="0.02">
-            <origin xyz="0 0 0" rpy="0 0 0"/>
-        </xacro:inertial_cylinder>
-    </link>
+                <cylinder radius="${wheel_r}" length="${wheel_l}"/>
+            </geometry>
+        </visual>
+        <collision>
+            <origin xyz="0 0 0" rpy="0 ${3.141/2} 0"/>
+            <geometry>
+                <cylinder radius="${wheel_r}" length="${wheel_l}"/>
+            </geometry>
+        </collision>
+        <xacro:inertial_cylinder mass="0.1" radius="${wheel_r}" length="${wheel_l}">
+            <origin xyz="0 0 0" rpy="0 0 0"/>
+        </xacro:inertial_cylinder>
+    </link>
+    <xacro:property name="wheel_mu" value="0.9"/>
+    <xacro:property name="wheel_mu2" value="0.2"/>
     <gazebo reference="back_right_wheel">
         <collision>
             <surface>
-                <friction>
-                    <ode>
-                        <mu>0.1</mu>
-                        <mu2>0.1</mu2>
+                <kp>1000000.0</kp>
+                <kd>100.0</kd>
+                <min_depth>0.01</min_depth>
+                <friction>
+                    <ode>
+                        <mu>${wheel_mu}</mu>
+                        <mu2>${wheel_mu2}</mu2>
+                        <fdir1>0 1.0 0</fdir1>
                     </ode>
                 </friction>
@@ -207,8 +215,12 @@
         <collision>
             <surface>
-                <friction>
-                    <ode>
-                        <mu>0.1</mu>
-                        <mu2>0.1</mu2>
+                <kp>1000000.0</kp>
+                <kd>100.0</kd>
+                <min_depth>0.01</min_depth>
+                <friction>
+                    <ode>
+                        <mu>${wheel_mu}</mu>
+                        <mu2>${wheel_mu2}</mu2>
+                        <fdir1>0 1.0 0</fdir1>
                     </ode>
                 </friction>
@@ -219,8 +231,12 @@
         <collision>
             <surface>
-                <friction>
-                    <ode>
-                        <mu>0.1</mu>
-                        <mu2>0.1</mu2>
+                <kp>1000000.0</kp>
+                <kd>100.0</kd>
+                <min_depth>0.01</min_depth>
+                <friction>
+                    <ode>
+                        <mu>${wheel_mu}</mu>
+                        <mu2>${wheel_mu2}</mu2>
+                        <fdir1>0 1.0 0</fdir1>
                     </ode>
                 </friction>
@@ -231,8 +247,12 @@
         <collision>
             <surface>
-                <friction>
-                    <ode>
-                        <mu>0.1</mu>
-                        <mu2>0.1</mu2>
+                <kp>1000000.0</kp>
+                <kd>100.0</kd>
+                <min_depth>0.01</min_depth>
+                <friction>
+                    <ode>
+                        <mu>${wheel_mu}</mu>
+                        <mu2>${wheel_mu2}</mu2>
+                        <fdir1>0 1.0 0</fdir1>
                     </ode>
                 </friction>
@@ -243,8 +263,12 @@
         <collision>
             <surface>
-                <friction>
-                    <ode>
-                        <mu>0.1</mu>
-                        <mu2>0.1</mu2>
+                <min_depth>0.01</min_depth>
+                <kp>1000000.0</kp>
+                <kd>100.0</kd>
+                <friction>
+                    <ode>
+                        <mu>${wheel_mu}</mu>
+                        <mu2>${wheel_mu2}</mu2>
+                        <fdir1>0 1.0 0</fdir1>
                     </ode>
                 </friction>
@@ -255,8 +279,12 @@
         <collision>
             <surface>
-                <friction>
-                    <ode>
-                        <mu>0.1</mu>
-                        <mu2>0.1</mu2>
+                <kp>1000000.0</kp>
+                <kd>100.0</kd>
+                <min_depth>0.01</min_depth>
+                <friction>
+                    <ode>
+                        <mu>${wheel_mu}</mu>
+                        <mu2>${wheel_mu2}</mu2>
+                        <fdir1>0 1.0 0</fdir1>
                     </ode>
                 </friction>
