Commit message: moved crawler package location

File: ws/src/crawler/description/robot_core.xacro (robot description, xacro)
@@ -30,7 +30,7 @@
             <geometry>
                 <!--
+                <mesh filename="package://crawler/meshes/chassis.dae" scale="1 1 1" />
+                -->
                 <box size="0.4 0.4 0.05"/>
-                -->`
-                <mesh filename="package://crawler/meshes/chassis.dae" scale="1 1 1" />
             </geometry>
             <material name="Gray">
@@ -339,3 +339,36 @@
         <origin xyz="0.1 0 0.1" rpy="0 0 0"/>
     </joint>
+    <link name="camera_link">
+        <visual>
+            <geometry>
+                <box size="0.1 0.1 0.1"/>
+            </geometry>
+        </visual>
+    </link>
+    <joint name="camera_joint" type="fixed">
+        <parent link="chassis"/>
+        <child link="camera_link"/>
+        <origin xyz="0.1 0 0.2" rpy="0 0 0"/>
+    </joint>
+    <gazebo reference="camera_link">
+      <sensor name="camera" type="depth">
+          <pose> 0 0 0 0 0 0 </pose>
+        <visualize>true</visualize>
+        <update_rate>10</update_rate>
+        <camera>
+            <horizontal_fov>1.089</horizontal_fov>
+            <image>
+                <format>R8G8B8</format>
+                <width>640</width>
+                <height>480</height>
+            </image>
+            <clip>
+                <near>0.05</near>
+                <far>8.0</far>
+            </clip>
+        </camera>
+    <plugin name="camera_controller" filename="libgazebo_ros_camera.so">
+    </plugin>
+    </sensor>
+    </gazebo>
 </robot>
